File: perimeter_leds.kicad_sch (KiCad schematic)
At the start: 22 parts

Commit message: progress
Parts:
- removed C1: 1uF, Capacitor_SMD:C_0805_2012Metric, symbol Device:C
- removed D1, D10, D11, D2, D3, D4, D5, D6, D7, D8, D9: WS2812B, LED_SMD:LED_WS2812B_PLCC4_5.0x5.0mm_P3.2mm, symbol LED:WS2812B
- added C12, C13, C14, C15, C16, C17, C18, C19, C20, C21, C22, C23, C24, C25, C26, C27, C28, C29, C30, C31, C32, C33, C34, C35, C36, C37, C38, C39, C40, C41, C42, C43, C44, C45, C46, C47, C48, C49, C50, C51, C52: 1uF, Capacitor_SMD:C_0603_1608Metric, symbol Device:C
- added D10, D11, D12, D13, D14, D15, D16, D17, D18, D19, D2, D20, D21, D22, D23, D24, D25, D26, D27, D28, D29, D3, D30, D31, D32, D33, D34, D35, D36, D37, D38, D39, D4, D40, D41, D42, D43, D44, D45, D46, D47, D48, D49, D5, D50, D51, D52, D6, D7, D8, D9: WS2812B-2020, LED_SMD:LED_WS2812B-2020_PLCC4_2.0x2.0mm, symbol LED:WS2812B-2020
- C10, C11, C2, C3, C4, C5, C6, C7, C8, C9: footprint Capacitor_SMD:C_0805_2012Metric -> Capacitor_SMD:C_0603_1608Metric
Connections:
- net 5V: now also C12.1, C13.1, C14.1, C15.1, C16.1, C17.1, C18.1, C19.1, C20.1, C21.1, C22.1, C23.1, C24.1, C25.1, C26.1, C27.1, C28.1, C29.1, C30.1, C31.1, C32.1, C33.1, C34.1, C35.1, C36.1, C37.1, C38.1, C39.1, C40.1, C41.1, C42.1, C43.1, C44.1, C45.1, C46.1, C47.1, C48.1, C49.1, C50.1, C51.1, C52.1, D10.4 (VDD), D11.4 (VDD), D12.4 (VDD), D13.4 (VDD), D14.4 (VDD), D15.4 (VDD), D16.4 (VDD), D17.4 (VDD), D18.4 (VDD), D19.4 (VDD), D2.4 (VDD), D20.4 (VDD), D21.4 (VDD), D22.4 (VDD), D23.4 (VDD), D24.4 (VDD), D25.4 (VDD), D26.4 (VDD), D27.4 (VDD), D28.4 (VDD), D29.4 (VDD), D3.4 (VDD), D30.4 (VDD), D31.4 (VDD), D32.4 (VDD), D33.4 (VDD), D34.4 (VDD), D35.4 (VDD), D36.4 (VDD), D37.4 (VDD), D38.4 (VDD), D39.4 (VDD), D4.4 (VDD), D40.4 (VDD), D41.4 (VDD), D42.4 (VDD), D43.4 (VDD), D44.4 (VDD), D45.4 (VDD), D46.4 (VDD), D47.4 (VDD), D48.4 (VDD), D49.4 (VDD), D5.4 (VDD), D50.4 (VDD), D51.4 (VDD), D52.4 (VDD), D6.4 (VDD), D7.4 (VDD), D8.4 (VDD), D9.4 (VDD)
- net DOUT: now also D40.1 (DOUT)
- net GND: now also C12.2, C13.2, C14.2, C15.2, C16.2, C17.2, C18.2, C19.2, C20.2, C21.2, C22.2, C23.2, C24.2, C25.2, C26.2, C27.2, C28.2, C29.2, C30.2, C31.2, C32.2, C33.2, C34.2, C35.2, C36.2, C37.2, C38.2, C39.2, C40.2, C41.2, C42.2, C43.2, C44.2, C45.2, C46.2, C47.2, C48.2, C49.2, C50.2, C51.2, C52.2, D10.2 (VSS), D11.2 (VSS), D12.2 (VSS), D13.2 (VSS), D14.2 (VSS), D15.2 (VSS), D16.2 (VSS), D17.2 (VSS), D18.2 (VSS), D19.2 (VSS), D2.2 (VSS), D20.2 (VSS), D21.2 (VSS), D22.2 (VSS), D23.2 (VSS), D24.2 (VSS), D25.2 (VSS), D26.2 (VSS), D27.2 (VSS), D28.2 (VSS), D29.2 (VSS), D3.2 (VSS), D30.2 (VSS), D31.2 (VSS), D32.2 (VSS), D33.2 (VSS), D34.2 (VSS), D35.2 (VSS), D36.2 (VSS), D37.2 (VSS), D38.2 (VSS), D39.2 (VSS), D4.2 (VSS), D40.2 (VSS), D41.2 (VSS), D42.2 (VSS), D43.2 (VSS), D44.2 (VSS), D45.2 (VSS), D46.2 (VSS), D47.2 (VSS), D48.2 (VSS), D49.2 (VSS), D5.2 (VSS), D50.2 (VSS), D51.2 (VSS), D52.2 (VSS), D6.2 (VSS), D7.2 (VSS), D8.2 (VSS), D9.2 (VSS)
- new net: D38.3 (DIN), D39.1 (DOUT)
- new net: D26.1 (DOUT), D39.3 (DIN)
- new net: D28.3 (DIN), D29.1 (DOUT)
- new net: D29.3 (DIN), D30.1 (DOUT)
- new net: D42.3 (DIN), D43.1 (DOUT)
- new net: D43.3 (DIN), D44.1 (DOUT)
- new net: D33.3 (DIN), D34.1 (DOUT)
- new net: D34.3 (DIN), D35.1 (DOUT)
- new net: D27.1 (DOUT), D52.3 (DIN)
- new net: D27.3 (DIN), D28.1 (DOUT)
- new net: D35.3 (DIN), D36.1 (DOUT)
- new net: D7.1 (DOUT), D8.3 (DIN)
- new net: D6.1 (DOUT), D7.3 (DIN)
- new net: D22.1 (DOUT), D23.3 (DIN)
- new net: D21.1 (DOUT), D22.3 (DIN)
- new net: D25.1 (DOUT), D26.3 (DIN)
- new net: D24.1 (DOUT), D25.3 (DIN)
- new net: D13.1 (DOUT), D14.3 (DIN)
- new net: D12.1 (DOUT), D13.3 (DIN)
- new net: D20.1 (DOUT), D21.3 (DIN)
- new net: D19.1 (DOUT), D20.3 (DIN)
- new net: D11.1 (DOUT), D12.3 (DIN)
- new net: D10.1 (DOUT), D11.3 (DIN)
- new net: D32.3 (DIN), D33.1 (DOUT)
- new net: D36.3 (DIN), D37.1 (DOUT)
- new net: D15.1 (DOUT), D16.3 (DIN)
- new net: D14.1 (DOUT), D15.3 (DIN)
- new net: D30.3 (DIN), D31.1 (DOUT)
- new net: D50.3 (DIN), D51.1 (DOUT)
- new net: D51.3 (DIN), D52.1 (DOUT)
- new net: D37.3 (DIN), D38.1 (DOUT)
- new net: D23.1 (DOUT), D24.3 (DIN)
- new net: D46.3 (DIN), D47.1 (DOUT)
- new net: D47.3 (DIN), D48.1 (DOUT)
- new net: D48.3 (DIN), D49.1 (DOUT)
- new net: D49.3 (DIN), D50.1 (DOUT)
- new net: D18.1 (DOUT), D19.3 (DIN)
- new net: D17.1 (DOUT), D18.3 (DIN)
- new net: D3.1 (DOUT), D4.3 (DIN)
- new net: D2.1 (DOUT), D3.3 (DIN)
- new net: D10.3 (DIN), D9.1 (DOUT)
- new net: D41.3 (DIN), D42.1 (DOUT)
- new net: D8.1 (DOUT), D9.3 (DIN)
- new net: D44.3 (DIN), D45.1 (DOUT)
- new net: D16.1 (DOUT), D17.3 (DIN)
- new net: D31.3 (DIN), D32.1 (DOUT)
- new net: D45.3 (DIN), D46.1 (DOUT)
- new net: D4.1 (DOUT), D5.3 (DIN)
- new net: D5.1 (DOUT), D6.3 (DIN)
- new net: D40.3 (DIN), D41.1 (DOUT)
Other:
- added sheet ws2812_and_cap (ws2812_and_cap.kicad_sch)
