File: YBF.kicad_sch (KiCad schematic)
At the start: 28 parts, among them J1 Chain_LED_out, J2 Chain_LED_return, SW1 1825910-6, SW2 1825910-6

Commit message: add fet
Parts:
- removed JP1: SolderJumper_3_Open, Jumper:SolderJumper-3_P1.3mm_Open_RoundedPad1.0x1.5mm_NumberLabels, symbol Jumper:SolderJumper_3_Open
- removed R1: 1M, Resistor_SMD:R_0603_1608Metric, symbol Device:R
- added TP1: DataChainOut, Connector_PinHeader_2.54mm:PinHeader_1x01_P2.54mm_Vertical, symbol Connector:TestPoint
- added TP2: ChainGND, Connector_PinHeader_2.54mm:PinHeader_1x01_P2.54mm_Vertical, symbol Connector:TestPoint
- added TP3: PerimGND, Connector_PinHeader_2.54mm:PinHeader_1x01_P2.54mm_Vertical, symbol Connector:TestPoint
- renumbered C4 to C2, C5 to C3, C2 to C4, C8 to C5, C3 to C8, H5 to H1, H6 to H2, H7 to H3, H3 to H4, H2 to H5, H4 to H6, SW2 to SW1, SW1 to SW2
Connections:
- net DATA_CHAIN_OUT: now also TP1.1
- net at J2.3 (Pin_3): now also J1.3 (Pin_3), MOSFET1.2 (D), TP2.1; no longer MOSFET2.2 (D)
- new net ws2812_and_cap69/GOUT: MOSFET2.2 (D), TP3.1
Other:
- removed sheet ws2812_and_cap
- added sheet ws2812_and_cap0 (ws2812_and_cap.kicad_sch)
- moved on the sheet: MOSFET2
