File: YBF.kicad_pcb (KiCad board)
At the start: 2 copper layers, 173.9 x 130.1 mm, 163 parts, among them J1 Chain_LED_out, J2 Chain_LED_return, SW1 1825910-6, SW2 1825910-6

Commit message: started on FETs
Parts:
- added H5: MountingHole, MountingHole:MountingHole_3mm, F.Cu at (144.5, 147.3)
- added MOSFET1: DMG2302UKQ-7, pfornage-kicad-lib:SOT23_DMG2302_DIO, F.Cu at (160.7, 124.4)
- added MOSFET2: DMG2302UKQ-7, pfornage-kicad-lib:SOT23_DMG2302_DIO, F.Cu at (120.8, 133.4)
- added R1: 1M, Resistor_SMD:R_0603_1608Metric, F.Cu at (114.8, 132.3)
- added R2: 10k, Resistor_SMD:R_0603_1608Metric, F.Cu at (115.1, 137.9)
- added R3: 10k, Resistor_SMD:R_0603_1608Metric, F.Cu at (116.9, 134.4)
- moved C11 12.4 mm to (115.8, 148.6)
- moved D3 12.3 mm to (118.2, 148.7)
- moved D2 6.48 mm to (123.4, 152.4)
- moved C10 6.48 mm to (121.2, 152.4)
- moved D1 6.19 mm to (129.6, 153.2)
- moved C9 6.15 mm to (127.3, 153.2)
- renumbered C4 to C2, C27 to C25, C25 to C26, C26 to C27, C5 to C3, C2 to C4, C43 to C41, C41 to C42, C42 to C43, C8 to C5, C75 to C73, C73 to C74, C74 to C75, C3 to C8, D19 to D17, D17 to D18, D18 to D19, D35 to D33, D33 to D34, D34 to D35, D67 to D65, D65 to D66, D66 to D67, H5 to H1, H6 to H2, H7 to H3, H3 to H4, H4 to H6, SW2 to SW1, SW1 to SW2
Connections:
- D1 pad 1: /ws2812_and_cap1/DOUT -> /ws2812_and_cap0/DOUT
- D1 pad 3: /ws2812_and_cap/DOUT -> PERIM_LED_DATA_IN
- D2 pad 1: /ws2812_and_cap2/DOUT -> /ws2812_and_cap1/DOUT
- D2 pad 3: /ws2812_and_cap1/DOUT -> /ws2812_and_cap0/DOUT
- D3 pad 1: /ws2812_and_cap/DOUT -> /ws2812_and_cap2/DOUT
- D3 pad 3: PERIM_LED_DATA_IN -> /ws2812_and_cap1/DOUT
- J1 pad 3: GND -> Net-(J1-Pin_3)
- J2 pad 3: GND -> Net-(J2-Pin_3)
Routing:
- net /ws2812_and_cap0/DOUT: track 0.00 -> 6.83 mm
- net /ws2812_and_cap/DOUT: track 6.83 -> 0.00 mm
